File: drv8212p_eval.kicad_pcb (KiCad board)
At the start: 2 copper layers, 46 x 26 mm, 23 parts, among them J1 Conn_01x06, J2 Conn_01x02, J3 Conn_01x02, U1 DRV8212P

Commit message: updated footprints
Parts:
- removed TP1: sense, TestPoint:TestPoint_Bridge_Pitch2.54mm_Drill1.0mm
- added J4: Conn_01x02, Connector_PinHeader_2.54mm:PinHeader_1x02_P2.54mm_Vertical, F.Cu at (131.3, 89.9)
- added kibuzzard-63E074E8: G***, kibuzzard-63E074E8, B.Cu at (144.8, 90.0)
- moved R1 3.14 mm to (130.0, 84.8), turned to 0 degrees
- moved kibuzzard-63D75466 0.30 mm to (130.0, 88.0)
Connections:
- net Net-(R1-Pad1) renamed /sense
Routing:
- net /sense: track 12.4 -> 9.33 mm
