File: drv8212p_eval.kicad_sch (KiCad schematic)
At the start: 13 parts, among them J1 Conn_01x06, J2 Conn_01x02, J3 Conn_01x02, U1 DRV8212P

Commit message: updated footprints
Parts:
- removed TP1: sense, TestPoint:TestPoint_Bridge_Pitch2.54mm_Drill1.0mm, symbol Connector:TestPoint
- added J?: Conn_01x02, Connector_PinHeader_2.54mm:PinHeader_1x02_P2.54mm_Vertical, symbol Connector_Generic:Conn_01x02
Connections:
- net GND: now also J?.1 (Pin_1)
- net sense: now reaches R1.1, U1.4 (GND)
- net sense: now also J?.2 (Pin_2)
Other:
- note added: "Sense Connector"
- moved on the sheet: H1, H2, H3, H4, J2
